File: Traffic lights/TrafficLights.brd (EAGLE design)
At the start: 46.4 x 55 mm, 29 parts, among them IC1 CPC1970, IC2 CPC1970, IC3 CPC1970, IC4 NE555, IC5 HEF4049B, J1 TB002-500-04BE, J2 PJ-037A, U1 SQ1922AEEH, U2 SQ1922AEEH, U3 CD4518BE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

Commit message: Fixed stuff
Parts:
- R13: device rcl:0207/2V -> rcl:R1206
- moved R12 66.7 mm to (35.0, 47.2)
- moved R13 61.8 mm to (33.0, 36.6), flipped to the bottom
- moved R11 48.9 mm to (41.0, 25.3)
- moved IC2 0.86 mm to (25.6, 43.6)
- moved C2 0.43 mm to (29.4, 13.0)
- moved J1 0.34 mm to (21.4, 51.4)
- moved R3 0.20 mm to (8.79, 8.32)
- moved R6 0.11 mm to (32.7, 37.9)
Connections:
- new net N$21: IC2.P$4, J1.2
- new net N$22: IC3.P$4, J1.1
- net VAC: no longer IC2.P$4, IC3.P$4, J1.1, J1.2
Routing:
- net N$22: track 0.00 -> 20.2 mm, vias 0 -> 2
- net VAC: track 47.2 -> 29.9 mm
- net VCC: track 9.77 -> 23.7 mm, vias 2 -> 12
- net N$21: track 0.00 -> 11.7 mm
- net N$2: track 30.7 -> 42.4 mm
- net GND: track 69.7 -> 61.9 mm, vias 15 -> 13
- net N$3: track 11.3 -> 18.9 mm, vias 1 -> 2
- net N$1: track 9.85 -> 14.1 mm
- net GREEN: track 27.4 -> 31.1 mm
- net N$18: track 9.37 -> 10.6 mm
- net YELLOW: track 26.7 -> 27.5 mm
- net N$9: track 44.7 -> 45.3 mm
- net AC_GND: track 31.6 -> 31.1 mm
- removed copper zone on layer 1, net VAC
